Commit message: removed unwanted!

File: src/kuka_allegro_description/urdf/allegro.urdf.xacro (robot description, xacro)
@@ -1,5 +1,4 @@
 <?xml version="1.0" ?>
 <robot xmlns:xacro="http://www.ros.org/wiki/xacro">
-  <xacro:include filename="$(find kuka_allegro_description)/urdf/allegro.transmission.xacro"/>
   <!-- ======================== BASE PARAMS ========================= -->
   <!-- ======================== FINGER PARAMS ======================== -->
@@ -20,10 +19,4 @@
     <color rgba="1 1 1 1"/>
   </material>
-  <xacro:macro name="allegro_macro" params="parent name *origin">
-    <joint name="${name}_base_joint" type="fixed">
-            <insert_block name="origin"/>
-            <parent link="${parent}"/>
-            <child link="allegro_mount"/>
-    </joint>
     <link name="allegro_mount">
     <inertial>
@@ -59,5 +52,5 @@
     <visual>
       <geometry>
-        <mesh filename="package://kuka_allegro_description/meshes/allegro/base_link_biotac.stl"/>
+        <mesh filename="package://kuka_allegro_description/meshes/allegro/base_link.stl"/>
       </geometry>
       <origin rpy="0 0 0" xyz="0 0 0 "/>
@@ -66,5 +59,5 @@
     <collision>
       <geometry>
-        <mesh filename="package://kuka_allegro_description/meshes/allegro/collision/base_link_biotac.stl"/>
+        <mesh filename="package://kuka_allegro_description/meshes/allegro/collision/base_link.stl"/>
       </geometry>
       <origin rpy="0 0 0" xyz="0 0 0 "/>
@@ -113,4 +106,5 @@
     <dynamics damping="1" friction="0"/>
   </joint>
+   <xacro:if value="$(arg include_part)">
   <!-- [LINK 1, 5, 9] -->
   <link name="index_link_1">
@@ -728,4 +722,4 @@
     <link name="thumb_link_3" servoP="1000" servoI="0" servoD="15"/>
   </klampt>
-</xacro:macro>
+</xacro:if>
 </robot>

File: src/kuka_allegro_description/urdf/kuka_allegro.xacro (robot description, xacro)
@@ -1,12 +1,23 @@
 <?xml version="1.0" ?>
 <robot name="kuka_allegro" xmlns:xacro="http://ros.org/wiki/xacro">
+<xacro:property name="M_PI"         value="3.1415926535897931"/>
+<xacro:arg name="include_part"    default="false" />
   <!-- kuka. It has already a world link. I do not need to make one.
   the default value for arg [name] is [iiwa]. Then the name of the EE will be [iiwa_link_ee] -->
  <xacro:include filename="$(find kuka_allegro_description)/urdf/iiwa14.urdf.xacro"/>
+ <!-- Include the KUKA mount -->
+<xacro:include filename="$(find kuka_allegro_description)/urdf/lbr4_mount.urdf.xacro"/>
+<xacro:lbr4_mount parent="iiwa_link_ee"/>
+    <joint name="lbr4_allegro" type="fixed">
+      <parent link="lbr4_mount"/>
+      <child link="allegro_mount"/>
+      <origin xyz="-0.0 0 0.01" rpy="0 1.57 0"/>
+    </joint>
+<!--    <xacro:include filename="$(find kuka_allegro_description)/urdf/allegro.transmission.xacro"/> -->
   <!-- allegro. [base_link] is the root for allegro hand  -->
  <xacro:include filename="$(find kuka_allegro_description)/urdf/allegro.urdf.xacro"/>
-<xacro:allegro_macro name="al" parent="iiwa_link_ee">
+<!-- <xacro:allegro_macro name="al" parent="iiwa_link_ee">
         <origin xyz="0 0 1" rpy="0 0 0" />
-</xacro:allegro_macro>
+</xacro:allegro_macro> -->
 <gazebo>
   <plugin name="gazebo_ros_control" filename="libgazebo_ros_control.so">

Commit message: modified gravity, fixed the inertia params

File: src/kuka_allegro_description/urdf/allegro.urdf.xacro (robot description, xacro)
@@ -92,5 +92,5 @@
       <mass value="0.0119" />
       <origin xyz="0 0 0" rpy="0 0 0"/>
-      <inertia ixx="1.01666658333e-06" ixy="0.0" ixz="0.0" iyy="6.47677333333e-07" iyz="0.0" izz="1.01666658333e-06" />
+      <inertia ixx="${stability_k*1.01666658333e-06}" ixy="0.0" ixz="0.0" iyy="${stability_k*6.47677333333e-07}" iyz="0.0" izz="${stability_k*1.01666658333e-06}" />
     </inertial>
   </link>
@@ -106,5 +106,4 @@
     <dynamics damping="1" friction="0"/>
   </joint>
-   <xacro:if value="$(arg include_part)">
   <!-- [LINK 1, 5, 9] -->
   <link name="index_link_1">
@@ -124,6 +123,6 @@
       <mass value="0.065" />
       <origin xyz="0 0 0" rpy="0 0 0"/>
-      <inertia ixx="7.95654166667e-05" ixy="1.7199e-05" ixz="8.75875e-06" iyy="2.47088833333e-05"
-	       iyz="2.413125e-05" izz="7.95654166667e-05" />
+      <inertia ixx="${stability_k*7.95654166667e-05}" ixy="${stability_k*1.7199e-05}" ixz="${stability_k*8.75875e-06}" iyy="${stability_k*2.47088833333e-05}"
+	       iyz="${stability_k*2.413125e-05}" izz="${stability_k*7.95654166667e-05}" />
     </inertial>
   </link>
@@ -156,6 +155,6 @@
       <mass value="0.0355" />
       <origin xyz="0 0 0" rpy="0 0 0"/>
-      <inertia ixx="2.63979183333e-05" ixy="6.67968e-06" ixz="4.783625e-06" iyy="1.34948516667e-05"
-	       iyz="9.372e-06" izz="2.63979183333e-05" />
+      <inertia ixx="${stability_k*2.63979183333e-05}" ixy="${stability_k*6.67968e-06}" ixz="${stability_k*4.783625e-06}" iyy="${stability_k*1.34948516667e-05}"
+	       iyz="${stability_k*9.372e-06}" izz="${stability_k*2.63979183333e-05}" />
     </inertial>
   </link>
@@ -188,6 +187,6 @@
       <mass value="0.0096" />
       <origin xyz="0 0 0" rpy="0 0 0"/>
-      <inertia ixx="4.701248e-06" ixy="1.255968e-06" ixz="1.2936e-06" iyy="3.649312e-06"
-	       iyz="1.7622e-06" izz="4.701248e-06" />
+      <inertia ixx="${stability_k1*4.701248e-06}" ixy="${stability_k1*1.255968e-06}" ixz="${stability_k1*1.2936e-06}" iyy="${stability_k1*3.649312e-06}"
+	       iyz="${stability_k1*1.7622e-06}" izz="${stability_k1*4.701248e-06}" />
     </inertial>
   </link>
@@ -219,5 +218,5 @@
       <mass value="0.0168" />
       <origin xyz="0 0 0" rpy="0 0 0"/>
-      <inertia ixx="9.68e-07" ixy="0" ixz="0" iyy="9.68e-07" iyz="0" izz="9.68e-07" />
+      <inertia ixx="${stability_k1*9.68e-07}" ixy="0" ixz="0" iyy="${stability_k1*9.68e-07}" iyz="0" izz="${stability_k1*.68e-07}" />
     </inertial>
   </link>
@@ -257,5 +256,5 @@
       <mass value="0.0119" />
       <origin xyz="0 0 0" rpy="0 0 0"/>
-      <inertia ixx="1.01666658333e-06" ixy="0.0" ixz="0.0" iyy="6.47677333333e-07" iyz="0.0" izz="1.01666658333e-06" />
+      <inertia ixx="${stability_k*1.01666658333e-06}" ixy="0.0" ixz="0.0" iyy="${stability_k*6.47677333333e-07}" iyz="0.0" izz="${stability_k*1.01666658333e-06}" />
     </inertial>
   </link>
@@ -288,6 +287,6 @@
       <mass value="0.065" />
       <origin xyz="0 0 0" rpy="0 0 0"/>
-      <inertia ixx="7.95654166667e-05" ixy="1.7199e-05" ixz="8.75875e-06" iyy="2.47088833333e-05"
-	       iyz="2.413125e-05" izz="7.95654166667e-05" />
+      <inertia ixx="${stability_k*7.95654166667e-05}" ixy="${stability_k*1.7199e-05}" ixz="${stability_k*8.75875e-06}" iyy="${stability_k*2.47088833333e-05}"
+	       iyz="${stability_k*2.413125e-05}" izz="${stability_k*7.95654166667e-05}" />
     </inertial>
   </link>
@@ -320,6 +319,6 @@
       <mass value="0.0355" />
       <origin xyz="0 0 0" rpy="0 0 0"/>
-      <inertia ixx="2.63979183333e-05" ixy="6.67968e-06" ixz="4.783625e-06" iyy="1.34948516667e-05"
-	       iyz="9.372e-06" izz="2.63979183333e-05" />
+      <inertia ixx="${stability_k*2.63979183333e-05}" ixy="${stability_k*6.67968e-06}" ixz="${stability_k*4.783625e-06}" iyy="${stability_k*1.34948516667e-05}"
+	       iyz="${stability_k*9.372e-06}" izz="${stability_k*2.63979183333e-05}" />
     </inertial>
   </link>
@@ -352,6 +351,6 @@
       <mass value="0.0096" />
       <origin xyz="0 0 0" rpy="0 0 0"/>
-      <inertia ixx="4.701248e-06" ixy="1.255968e-06" ixz="1.2936e-06" iyy="3.649312e-06"
-	       iyz="1.7622e-06" izz="4.701248e-06" />
+      <inertia ixx="${stability_k1*4.701248e-06}" ixy="${stability_k1*1.255968e-06}" ixz="${stability_k1*1.2936e-06}" iyy="${stability_k1*3.649312e-06}"
+	       iyz="${stability_k1*1.7622e-06}" izz="${stability_k1*4.701248e-06}" />
     </inertial>
   </link>
@@ -383,5 +382,5 @@
       <mass value="0.0168" />
       <origin xyz="0 0 0" rpy="0 0 0"/>
-      <inertia ixx="9.68e-07" ixy="0" ixz="0" iyy="9.68e-07" iyz="0" izz="9.68e-07" />
+      <inertia ixx="${stability_k1*9.68e-07}" ixy="0" ixz="0" iyy="${stability_k1*9.68e-07}" iyz="0" izz="${stability_k1*9.68e-07}" />
     </inertial>
   </link>
@@ -408,5 +407,5 @@
       <mass value="0.0119" />
       <origin xyz="0 0 0" rpy="0 0 0"/>
-      <inertia ixx="1.01666658333e-06" ixy="0.0" ixz="0.0" iyy="6.47677333333e-07" iyz="0.0" izz="1.01666658333e-06" />
+      <inertia ixx="${stability_k*1.01666658333e-06}" ixy="0.0" ixz="0.0" iyy="${stability_k*6.47677333333e-07}" iyz="0.0" izz="${stability_k*1.01666658333e-06}" />
     </inertial>
   </link>
@@ -439,6 +438,6 @@
       <mass value="0.065" />
       <origin xyz="0 0 0" rpy="0 0 0"/>
-      <inertia ixx="7.95654166667e-05" ixy="1.7199e-05" ixz="8.75875e-06" iyy="2.47088833333e-05"
-	       iyz="2.413125e-05" izz="7.95654166667e-05" />
+      <inertia ixx="${stability_k*7.95654166667e-05}" ixy="${stability_k*1.7199e-05}" ixz="${stability_k*8.75875e-06}" iyy="${stability_k*2.47088833333e-05}"
+	       iyz="${stability_k*2.413125e-05}" izz="${stability_k*7.95654166667e-05}" />
     </inertial>
   </link>
@@ -471,6 +470,6 @@
       <mass value="0.0355" />
       <origin xyz="0 0 0" rpy="0 0 0"/>
-      <inertia ixx="2.63979183333e-05" ixy="6.67968e-06" ixz="4.783625e-06" iyy="1.34948516667e-05"
-	       iyz="9.372e-06" izz="2.63979183333e-05" />
+      <inertia ixx="${stability_k*2.63979183333e-05}" ixy="${stability_k*6.67968e-06}" ixz="${stability_k*4.783625e-06}" iyy="${stability_k*1.34948516667e-05}"
+	       iyz="${stability_k*9.372e-06}" izz="${stability_k*2.63979183333e-05}" />
     </inertial>
   </link>
@@ -503,6 +502,6 @@
       <mass value="0.0096" />
       <origin xyz="0 0 0" rpy="0 0 0"/>
-      <inertia ixx="4.701248e-06" ixy="1.255968e-06" ixz="1.2936e-06" iyy="3.649312e-06"
-	       iyz="1.7622e-06" izz="4.701248e-06" />
+      <inertia ixx="${stability_k1*4.701248e-06}" ixy="${stability_k1*1.255968e-06}" ixz="${stability_k1*1.2936e-06}" iyy="${stability_k1*3.649312e-06}"
+	       iyz="${stability_k1*1.7622e-06}" izz="${stability_k1*4.701248e-06}" />
     </inertial>
   </link>
@@ -534,5 +533,5 @@
       <mass value="0.0168" />
       <origin xyz="0 0 0" rpy="0 0 0"/>
-      <inertia ixx="9.68e-07" ixy="0" ixz="0" iyy="9.68e-07" iyz="0" izz="9.68e-07" />
+      <inertia ixx="${stability_k1*9.68e-07}" ixy="0" ixz="0" iyy="${stability_k1*9.68e-07}" iyz="0" izz="${stability_k1*9.68e-07}" />
     </inertial>
   </link>
@@ -560,6 +559,6 @@
       <mass value="0.0176" />
       <origin xyz="0 0 0" rpy="0 0 0"/>
-      <inertia ixx="1.89273333333e-5" ixy="7.16716e-06" ixz="5.35568e-06" iyy="1.43008213333e-05"
-	       iyz="6.8068e-06" izz="1.89273333333e-05" />
+      <inertia ixx="${stability_k*1.89273333333e-5}" ixy="${stability_k*7.16716e-06}" ixz="${stability_k*5.35568e-06}" iyy="${stability_k*1.43008213333e-05}"
+	       iyz="${stability_k*6.8068e-06}" izz="${stability_k*1.89273333333e-05}" />
     </inertial>
   </link>
@@ -593,6 +592,6 @@
       <mass value="0.0119" />
       <origin xyz="0 0 0" rpy="0 0 0"/>
-      <inertia ixx="4.24250866667e-06" ixy="1.032087e-06" ixz="1.603525e-06" iyy="4.52362633333e-06"
-	       iyz="1.44808125e-06" izz="4.24250866667e-06" />
+      <inertia ixx="${stability_k*4.24250866667e-06}" ixy="${stability_k*1.032087e-06}" ixz="${stability_k*1.603525e-06}" iyy="${stability_k*4.52362633333e-06}"
+	       iyz="${stability_k*1.44808125e-06}" izz="${stability_k*4.24250866667e-06}" />
     </inertial>
   </link>
@@ -626,6 +625,6 @@
       <mass value="0.038" />
       <origin xyz="0 0 0" rpy="0 0 0"/>
-      <inertia ixx="4.30439933333e-05" ixy="9.57068e-06" ixz="5.1205e-06" iyy="1.44451933333e-05"
-	       iyz="1.342825e-05" izz="4.30439933333e-05" />
+      <inertia ixx="${stability_k*4.30439933333e-05}" ixy="${stability_k*9.57068e-06}" ixz="${stability_k*5.1205e-06}" iyy="${stability_k*1.44451933333e-05}"
+	       iyz="${stability_k*1.342825e-05}" izz="${stability_k*4.30439933333e-05}" />
     </inertial>
   </link>
@@ -659,6 +658,6 @@
       <mass value="0.0388" />
       <origin xyz="0 0 0" rpy="0 0 0"/>
-      <inertia ixx="3.29223173333e-05" ixy="8.042076e-06" ixz="5.2283e-06" iyy="1.47493026667e-5"
-	       iyz="1.1283525e-5" izz="3.29223173333e-05" />
+      <inertia ixx="${stability_k1*3.29223173333e-05}" ixy="${stability_k1*8.042076e-06}" ixz="${stability_k1*5.2283e-06}" iyy="${stability_k1*1.47493026667e-5}"
+	       iyz="${stability_k1*1.1283525e-5}" izz="${stability_k1*3.29223173333e-05}" />
     </inertial>
   </link>
@@ -691,5 +690,5 @@
       <mass value="0.0168" />
       <origin xyz="0 0 0" rpy="0 0 0"/>
-      <inertia ixx="9.68e-07" ixy="0" ixz="0" iyy="9.68e-07" iyz="0" izz="9.68e-07" />
+      <inertia ixx="${stability_k1*9.68e-07}" ixy="0" ixz="0" iyy="${stability_k1*9.68e-07}" iyz="0" izz="${stability_k1*9.68e-07}" />
     </inertial>
   </link>
@@ -722,4 +721,5 @@
     <link name="thumb_link_3" servoP="1000" servoI="0" servoD="15"/>
   </klampt>
+<xacro:if value="$(arg include_part)">
 </xacro:if>
 </robot>

File: src/kuka_allegro_description/urdf/kuka_allegro.xacro (robot description, xacro)
@@ -2,4 +2,6 @@
 <robot name="kuka_allegro" xmlns:xacro="http://ros.org/wiki/xacro">
 <xacro:property name="M_PI"         value="3.1415926535897931"/>
+<xacro:property name="stability_k"         value="1e3"/>
+<xacro:property name="stability_k1"         value="1e4"/>
 <xacro:arg name="include_part"    default="false" />
   <!-- kuka. It has already a world link. I do not need to make one.
@@ -12,7 +14,7 @@
       <parent link="lbr4_mount"/>
       <child link="allegro_mount"/>
-      <origin xyz="-0.0 0 0.01" rpy="0 1.57 0"/>
+      <origin xyz="-0.0 0 0.01" rpy="0 1.57 3.14"/>
     </joint>
-<!--    <xacro:include filename="$(find kuka_allegro_description)/urdf/allegro.transmission.xacro"/> -->
+   <xacro:include filename="$(find kuka_allegro_description)/urdf/allegro.transmission.xacro"/>
   <!-- allegro. [base_link] is the root for allegro hand  -->
  <xacro:include filename="$(find kuka_allegro_description)/urdf/allegro.urdf.xacro"/>
